File: Wsprry-Pi-LPF/Wsprry-Pi-LPF.kicad_sch (KiCad schematic)
At the start: 13 parts, among them J1 Conn_01x04, J2 Conn_01x04

Commit message: Enlarge axial L pad, add Toroid co-pad
Parts:
- L2, L4, L6: footprint Inductor_THT:L_Axial_L5.3mm_D2.2mm_P7.62mm_Horizontal_Vishay_IM-1 -> Wsprry Pi LPF:L_Axial_Horiz_Torroid_Vert_12mm_D5mm_P10.2mm
Changed lines of the file:
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@@
 			)
 		)
-		(property "Footprint" "Inductor_THT:L_Axial_L5.3mm_D2.2mm_P7.62mm_Horizontal_Vishay_IM-1"
+		(property "Footprint" "Wsprry Pi LPF:L_Axial_Horiz_Torroid_Vert_12mm_D5mm_P10.2mm"
 			(at 171.45 107.95 0)
 			(effects
@@
 			)
 		)
-		(property "Footprint" "Inductor_THT:L_Axial_L5.3mm_D2.2mm_P7.62mm_Horizontal_Vishay_IM-1"
+		(property "Footprint" "Wsprry Pi LPF:L_Axial_Horiz_Torroid_Vert_12mm_D5mm_P10.2mm"
 			(at 130.81 107.95 0)
 			(effects
@@
 			)
 		)
-		(property "Footprint" "Inductor_THT:L_Axial_L5.3mm_D2.2mm_P7.62mm_Horizontal_Vishay_IM-1"
+		(property "Footprint" "Wsprry Pi LPF:L_Axial_Horiz_Torroid_Vert_12mm_D5mm_P10.2mm"
 			(at 151.13 107.95 0)
 			(effects
